File: KiCad Numpad/New Project-backups/KiCad NumpadHS.kicad_pcb (KiCad board)
At the start: 2 copper layers, 100 x 98.4 mm, 37 parts, among them U1 Arduino_Pro_Micro

Commit message: PCB Layout Complete
Parts:
- turned S3 to 180 degrees
Routing:
- net COL3: track 129.2 -> 124.3 mm
- net ROW5: track 144.9 -> 141.4 mm
- net COL1: track 167.2 -> 165.9 mm
