File: KiCad Numpad/KiCad Numpad.kicad_sch (KiCad schematic)
At the start: 36 parts, among them U1 ProMicro

Commit message: 1
Other:
- moved on the sheet: U1
Changed lines of the file:
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@@
 		)
 		(instances
-			(project "New Project"
+			(project "KiCad Numpad"
 				(path "/399776d7-afe2-437e-8a47-9123c5af5dd7"
 					(reference "D13")
@@
 		)
 		(instances
-			(project "New Project"
+			(project "KiCad Numpad"
 				(path "/399776d7-afe2-437e-8a47-9123c5af5dd7"
 					(reference "D3")
@@
 		)
 		(instances
-			(project "New Project"
+			(project "KiCad Numpad"
 				(path "/399776d7-afe2-437e-8a47-9123c5af5dd7"
 					(reference "MX1")
@@
 		)
 		(instances
-			(project "New Project"
+			(project "KiCad Numpad"
 				(path "/399776d7-afe2-437e-8a47-9123c5af5dd7"
 					(reference "MX15")
@@
 		)
 		(instances
-			(project "New Project"
+			(project "KiCad Numpad"
 				(path "/399776d7-afe2-437e-8a47-9123c5af5dd7"
 					(reference "D5")
@@
 		)
 		(instances
-			(project "New Project"
+			(project "KiCad Numpad"
 				(path "/399776d7-afe2-437e-8a47-9123c5af5dd7"
 					(reference "MX17")
@@
 		)
 		(instances
-			(project "New Project"
+			(project "KiCad Numpad"
 				(path "/399776d7-afe2-437e-8a47-9123c5af5dd7"
 					(reference "S3")
@@
 		)
 		(instances
-			(project "New Project"
+			(project "KiCad Numpad"
 				(path "/399776d7-afe2-437e-8a47-9123c5af5dd7"
 					(reference "MX14")
@@
 		)
 		(instances
-			(project "New Project"
+			(project "KiCad Numpad"
 				(path "/399776d7-afe2-437e-8a47-9123c5af5dd7"
 					(reference "D10")
@@
 		)
 		(instances
-			(project "New Project"
+			(project "KiCad Numpad"
 				(path "/399776d7-afe2-437e-8a47-9123c5af5dd7"
 					(reference "D2")
@@
 		)
 		(instances
-			(project "New Project"
+			(project "KiCad Numpad"
 				(path "/399776d7-afe2-437e-8a47-9123c5af5dd7"
 					(reference "MX12")
@@
 		)
 		(instances
-			(project "New Project"
+			(project "KiCad Numpad"
 				(path "/399776d7-afe2-437e-8a47-9123c5af5dd7"
 					(reference "D16")
@@
 		)
 		(instances
-			(project "New Project"
+			(project "KiCad Numpad"
 				(path "/399776d7-afe2-437e-8a47-9123c5af5dd7"
 					(reference "MX13")
@@
 		)
 		(instances
-			(project "New Project"
+			(project "KiCad Numpad"
 				(path "/399776d7-afe2-437e-8a47-9123c5af5dd7"
 					(reference "D17")
@@
 		)
 		(instances
-			(project "New Project"
+			(project "KiCad Numpad"
 				(path "/399776d7-afe2-437e-8a47-9123c5af5dd7"
 					(reference "MX7")
@@
 		)
 		(instances
-			(project "New Project"
+			(project "KiCad Numpad"
 				(path "/399776d7-afe2-437e-8a47-9123c5af5dd7"
 					(reference "D1")
@@
 		)
 		(instances
-			(project "New Project"
+			(project "KiCad Numpad"
 				(path "/399776d7-afe2-437e-8a47-9123c5af5dd7"
 					(reference "MX10")
@@
 		)
 		(instances
-			(project "New Project"
+			(project "KiCad Numpad"
 				(path "/399776d7-afe2-437e-8a47-9123c5af5dd7"
 					(reference "D11")
@@
 		)
 		(instances
-			(project "New Project"
+			(project "KiCad Numpad"
 				(path "/399776d7-afe2-437e-8a47-9123c5af5dd7"
 					(reference "MX2")
@@
 		)
 		(instances
-			(project "New Project"
+			(project "KiCad Numpad"
 				(path "/399776d7-afe2-437e-8a47-9123c5af5dd7"
 					(reference "D4")
@@
 		)
 		(instances
-			(project "New Project"
+			(project "KiCad Numpad"
 				(path "/399776d7-afe2-437e-8a47-9123c5af5dd7"
 					(reference "S2")
@@
 		)
 		(instances
-			(project "New Project"
+			(project "KiCad Numpad"
 				(path "/399776d7-afe2-437e-8a47-9123c5af5dd7"
 					(reference "D6")
@@
 		)
 		(instances
-			(project "New Project"
+			(project "KiCad Numpad"
 				(path "/399776d7-afe2-437e-8a47-9123c5af5dd7"
 					(reference "D15")
@@
 		)
 		(instances
-			(project "New Project"
+			(project "KiCad Numpad"
 				(path "/399776d7-afe2-437e-8a47-9123c5af5dd7"
 					(reference "S1")
@@
 		)
 		(instances
-			(project "New Project"
+			(project "KiCad Numpad"
 				(path "/399776d7-afe2-437e-8a47-9123c5af5dd7"
 					(reference "D14")
@@
 		)
 		(instances
-			(project "New Project"
+			(project "KiCad Numpad"
 				(path "/399776d7-afe2-437e-8a47-9123c5af5dd7"
 					(reference "MX16")
@@
 		)
 		(instances
-			(project "New Project"
+			(project "KiCad Numpad"
 				(path "/399776d7-afe2-437e-8a47-9123c5af5dd7"
 					(reference "MX5")
@@
 		)
 		(instances
-			(project "New Project"
+			(project "KiCad Numpad"
 				(path "/399776d7-afe2-437e-8a47-9123c5af5dd7"
 					(reference "MX3")
@@
 		)
 		(instances
-			(project "New Project"
+			(project "KiCad Numpad"
 				(path "/399776d7-afe2-437e-8a47-9123c5af5dd7"
 					(reference "D7")
@@
 		)
 		(instances
-			(project "New Project"
+			(project "KiCad Numpad"
 				(path "/399776d7-afe2-437e-8a47-9123c5af5dd7"
 					(reference "MX4")
@@
 		)
 		(instances
-			(project "New Project"
+			(project "KiCad Numpad"
 				(path "/399776d7-afe2-437e-8a47-9123c5af5dd7"
 					(reference "MX11")
@@
 		)
 		(instances
-			(project "New Project"
+			(project "KiCad Numpad"
 				(path "/399776d7-afe2-437e-8a47-9123c5af5dd7"
 					(reference "D12")
@@
 		)
 		(instances
-			(project "New Project"
+			(project "KiCad Numpad"
 				(path "/399776d7-afe2-437e-8a47-9123c5af5dd7"
 					(reference "MX9")
@@
 		)
 		(instances
-			(project "New Project"
+			(project "KiCad Numpad"
 				(path "/399776d7-afe2-437e-8a47-9123c5af5dd7"
 					(reference "D9")
@@
 		)
 		(instances
-			(project "New Project"
+			(project "KiCad Numpad"
 				(path "/399776d7-afe2-437e-8a47-9123c5af5dd7"
 					(reference "MX6")
@@
 	(symbol
 		(lib_id "PCM_marbastlib-promicroish:Arduino_ProMicro")
-		(at 77.47 102.87 0)
+		(at 77.47 93.98 0)
 		(unit 1)
 		(exclude_from_sim no)
@@
 		(fields_autoplaced yes)
 		(property "Reference" "U1"
-			(at 77.47 81.28 0)
+			(at 77.47 72.39 0)
 			(effects
 				(font
@@
 		)
 		(property "Value" "ProMicro"
-			(at 77.47 83.82 0)
+			(at 77.47 74.93 0)
 			(effects
 				(font
@@
 		)
 		(property "Footprint" "PCM_marbastlib-xp-promicroish:ProMicro_USBup"
-			(at 77.47 133.35 0)
+			(at 77.47 124.46 0)
 			(effects
 				(font
@@
 		)
 		(property "Datasheet" ""
-			(at 64.77 88.9 0)
+			(at 64.77 80.01 0)
 			(effects
 				(font
@@
 		)
 		(property "Description" "Symbol for an Arduino Pro Micro"
-			(at 77.47 102.87 0)
+			(at 77.47 93.98 0)
 			(effects
 				(font
@@
 		)
 		(instances
-			(project "New Project"
+			(project "KiCad Numpad"
 				(path "/399776d7-afe2-437e-8a47-9123c5af5dd7"
 					(reference "U1")

Commit message: push2
Parts:
- removed S1: MX_stab, PCM_marbastlib-mx:STAB_MX_2u, symbol PCM_marbastlib-mx:MX_stab
- removed U1: ProMicro, PCM_marbastlib-xp-promicroish:ProMicro_USBup, symbol PCM_marbastlib-promicroish:Arduino_ProMicro
- added D8: D_Small, Diode_SMD:D_SOD-123, symbol Device:D_Small
- added MX8: MX_SW_solder, PCM_marbastlib-mx:SW_MX_1u, symbol PCM_marbastlib-mx:MX_SW_solder
- added U1: Arduino_Pro_Micro, ScottoKeebs_MCU:Arduino_Pro_Micro, symbol ScottoKeebs:MCU_Arduino_Pro_Micro
Connections:
- net COL1: now also U1.5 (2/PD1)
- net COL2: now also U1.6 (3/PD0)
- net COL3: now also U1.7 (4/PD4)
- net COL4: now also MX8.1, U1.8 (5/PC6)
- net ROW1: now also U1.9 (6/PD7)
- net ROW2: now also U1.10 (7/PE6)
- net ROW3: now also D8.1 (K), U1.11 (8/PB4)
- net ROW4: now also U1.12 (9/PB5); no longer D3.1 (K)
- net ROW5: now also D3.1 (K), U1.20 (A3/PF4)
- new net: D8.2 (A), MX8.2
- new net GND: U1.23 (GND), U1.3 (GND), U1.4 (GND)
Other:
- moved on the sheet: D12, D3, MX12, MX3

Commit message: update
Connections:
- net COL2: no longer MX16.1
- net COL3: now also MX16.1
- removed net GND: U1.23 (GND), U1.3 (GND), U1.4 (GND)
Other:
- moved on the sheet: D16, MX16

Commit message: PCB Layout Complete
Parts:
- MX1, MX10, MX11, MX12, MX13, MX14, MX15, MX16, MX17, MX3, MX5, MX6, MX7, MX8, MX9: footprint PCM_marbastlib-mx:SW_MX_1u -> PCM_marbastlib-mx:SW_MX_HS_CPG151101S11_1u
- MX2, MX4: footprint PCM_marbastlib-mx:SW_MX_1.5u -> PCM_marbastlib-mx:SW_MX_HS_CPG151101S11_1.5u
Changed lines of the file:
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@@
 			)
 		)
-		(property "Footprint" "PCM_marbastlib-mx:SW_MX_1u"
+		(property "Footprint" "PCM_marbastlib-mx:SW_MX_HS_CPG151101S11_1u"
 			(at 127 63.5 0)
 			(effects
@@
 			)
 		)
-		(property "Footprint" "PCM_marbastlib-mx:SW_MX_1u"
+		(property "Footprint" "PCM_marbastlib-mx:SW_MX_HS_CPG151101S11_1u"
 			(at 152.4 101.6 0)
 			(effects
@@
 			)
 		)
-		(property "Footprint" "PCM_marbastlib-mx:SW_MX_1u"
+		(property "Footprint" "PCM_marbastlib-mx:SW_MX_HS_CPG151101S11_1u"
 			(at 127 114.3 0)
 			(effects
@@
 			)
 		)
-		(property "Footprint" "PCM_marbastlib-mx:SW_MX_1u"
+		(property "Footprint" "PCM_marbastlib-mx:SW_MX_HS_CPG151101S11_1u"
 			(at 139.7 101.6 0)
 			(effects
@@
 			)
 		)
-		(property "Footprint" "PCM_marbastlib-mx:SW_MX_1u"
+		(property "Footprint" "PCM_marbastlib-mx:SW_MX_HS_CPG151101S11_1u"
 			(at 160.02 76.2 0)
 			(effects
@@
 			)
 		)
-		(property "Footprint" "PCM_marbastlib-mx:SW_MX_1u"
+		(property "Footprint" "PCM_marbastlib-mx:SW_MX_HS_CPG151101S11_1u"
 			(at 127 101.6 0)
 			(effects
@@
 			)
 		)
-		(property "Footprint" "PCM_marbastlib-mx:SW_MX_1u"
+		(property "Footprint" "PCM_marbastlib-mx:SW_MX_HS_CPG151101S11_1u"
 			(at 152.4 76.2 0)
 			(effects
@@
 			)
 		)
-		(property "Footprint" "PCM_marbastlib-mx:SW_MX_1u"
+		(property "Footprint" "PCM_marbastlib-mx:SW_MX_HS_CPG151101S11_1u"
 			(at 139.7 88.9 0)
 			(effects
@@
 			)
 		)
-		(property "Footprint" "PCM_marbastlib-mx:SW_MX_1u"
+		(property "Footprint" "PCM_marbastlib-mx:SW_MX_HS_CPG151101S11_1u"
 			(at 160.02 88.9 0)
 			(effects
@@
 			)
 		)
-		(property "Footprint" "PCM_marbastlib-mx:SW_MX_1.5u"
+		(property "Footprint" "PCM_marbastlib-mx:SW_MX_HS_CPG151101S11_1.5u"
 			(at 143.51 63.5 0)
 			(effects
@@
 			)
 		)
-		(property "Footprint" "PCM_marbastlib-mx:SW_MX_1u"
+		(property "Footprint" "PCM_marbastlib-mx:SW_MX_HS_CPG151101S11_1u"
 			(at 152.4 114.3 0)
 			(effects
@@
 			)
 		)
-		(property "Footprint" "PCM_marbastlib-mx:SW_MX_1u"
+		(property "Footprint" "PCM_marbastlib-mx:SW_MX_HS_CPG151101S11_1u"
 			(at 127 76.2 0)
 			(effects
@@
 			)
 		)
-		(property "Footprint" "PCM_marbastlib-mx:SW_MX_1u"
+		(property "Footprint" "PCM_marbastlib-mx:SW_MX_HS_CPG151101S11_1u"
 			(at 160.02 109.22 0)
 			(effects
@@
 			)
 		)
-		(property "Footprint" "PCM_marbastlib-mx:SW_MX_1.5u"
+		(property "Footprint" "PCM_marbastlib-mx:SW_MX_HS_CPG151101S11_1.5u"
 			(at 160.02 63.5 0)
 			(effects
@@
 			)
 		)
-		(property "Footprint" "PCM_marbastlib-mx:SW_MX_1u"
+		(property "Footprint" "PCM_marbastlib-mx:SW_MX_HS_CPG151101S11_1u"
 			(at 152.4 88.9 0)
 			(effects
@@
 			)
 		)
-		(property "Footprint" "PCM_marbastlib-mx:SW_MX_1u"
+		(property "Footprint" "PCM_marbastlib-mx:SW_MX_HS_CPG151101S11_1u"
 			(at 127 88.9 0)
 			(effects
@@
 			)
 		)
-		(property "Footprint" "PCM_marbastlib-mx:SW_MX_1u"
+		(property "Footprint" "PCM_marbastlib-mx:SW_MX_HS_CPG151101S11_1u"
 			(at 139.7 76.2 0)
 			(effects

Commit message: Placing Order #1
Parts:
- added H1, H2, H3, H4: MountingHole, MountingHole:MountingHole_2.2mm_M2, symbol Mechanical:MountingHole
- MX1, MX10, MX11, MX12, MX13, MX14, MX15, MX16, MX17, MX3, MX5, MX6, MX7, MX8, MX9: footprint PCM_marbastlib-mx:SW_MX_HS_CPG151101S11_1u -> PCM_marbastlib-mx:SW_MX_1u
- MX2, MX4: footprint PCM_marbastlib-mx:SW_MX_HS_CPG151101S11_1.5u -> PCM_marbastlib-mx:SW_MX_1.5u
Connections:
- net COL4 is gone; now on net COL3: MX12.1, MX3.1, MX4.1, MX8.1, U1.8 (5/PC6)
- net ROW5 is gone; now on net ROW4: D16.1 (K), D17.1 (K), D3.1 (K), U1.20 (A3/PF4)
- net COL1: now also MX10.1, MX14.1, MX2.1, MX6.1, U1.6 (3/PD0); no longer MX1.1, MX13.1, MX17.1, MX5.1, MX9.1, U1.5 (2/PD1)
- net COL2: now also MX11.1, MX15.1, MX16.1, MX7.1, U1.7 (4/PD4); no longer MX10.1, MX14.1, MX2.1, MX6.1, U1.6 (3/PD0)
- net COL3: no longer MX11.1, MX15.1, MX16.1, MX7.1, U1.7 (4/PD4)
- net ROW1: now also D12.1 (K), D5.1 (K), D6.1 (K), D7.1 (K), U1.10 (7/PE6); no longer D1.1 (K), D2.1 (K), D4.1 (K), U1.9 (6/PD7)
- net ROW2: now also D10.1 (K), D11.1 (K), D8.1 (K), D9.1 (K), U1.11 (8/PB4); no longer D12.1 (K), D5.1 (K), D6.1 (K), D7.1 (K), U1.10 (7/PE6)
- net ROW3: now also D13.1 (K), D14.1 (K), D15.1 (K), U1.12 (9/PB5); no longer D10.1 (K), D11.1 (K), D8.1 (K), D9.1 (K), U1.11 (8/PB4)
- net ROW4: no longer D13.1 (K), D14.1 (K), D15.1 (K), U1.12 (9/PB5)
- new net COL0: MX1.1, MX13.1, MX17.1, MX5.1, MX9.1, U1.5 (2/PD1)
- new net ROW0: D1.1 (K), D2.1 (K), D4.1 (K), U1.9 (6/PD7)
Other:
- moved on the sheet: U1
